File: pcb/HeadPower.sch (KiCad schematic (older format))
At the start: 9 parts

Commit message: Adds more to the schematic
Parts:
- C? (x4): footprint (none) -> Capacitor_SMD:C_0805_2012Metric
- J?, SW?: footprint (none) -> Connector_PinHeader_2.54mm:PinHeader_1x02_P2.54mm_Vertical
Changed lines of the file:
@@
 $Descr A4 11693 8268
 encoding utf-8
-Sheet 2 3
+Sheet 2 14
 Title ""
 Date ""
@@
 F 0 "C?" H 3965 3146 50  0000 L CNN
 F 1 "10μF" H 3965 3055 50  0000 L CNN
-F 2 "" H 3888 2950 50  0001 C CNN
+F 2 "Capacitor_SMD:C_0805_2012Metric" H 3888 2950 50  0001 C CNN
 F 3 "~" H 3850 3100 50  0001 C CNN
 	1    3850 3100
@@
 F 0 "C?" H 5215 3146 50  0000 L CNN
 F 1 "22μF" H 5215 3055 50  0000 L CNN
-F 2 "" H 5138 2950 50  0001 C CNN
+F 2 "Capacitor_SMD:C_0805_2012Metric" H 5138 2950 50  0001 C CNN
 F 3 "~" H 5100 3100 50  0001 C CNN
 	1    5100 3100
@@
 F 0 "C?" H 5765 3146 50  0000 L CNN
 F 1 "1μF" H 5765 3055 50  0000 L CNN
-F 2 "" H 5688 2950 50  0001 C CNN
+F 2 "Capacitor_SMD:C_0805_2012Metric" H 5688 2950 50  0001 C CNN
 F 3 "~" H 5650 3100 50  0001 C CNN
 	1    5650 3100
@@
 F 0 "C?" H 6665 3146 50  0000 L CNN
 F 1 "1μF" H 6665 3055 50  0000 L CNN
-F 2 "" H 6588 2950 50  0001 C CNN
+F 2 "Capacitor_SMD:C_0805_2012Metric" H 6588 2950 50  0001 C CNN
 F 3 "~" H 6550 3100 50  0001 C CNN
 	1    6550 3100
@@
 F 0 "J?" H 2507 2467 50  0000 C CNN
 F 1 "Barrel_Jack_Switch_Pin3Ring" H 2507 2376 50  0000 C CNN
-F 2 "" H 2500 2110 50  0001 C CNN
+F 2 "Connector_PinHeader_2.54mm:PinHeader_1x02_P2.54mm_Vertical" H 2500 2110 50  0001 C CNN
 F 3 "~" H 2500 2110 50  0001 C CNN
 	1    2450 2150
@@
 F 0 "SW?" H 3450 2985 50  0000 C CNN
 F 1 "SW_SPST" H 3450 2894 50  0000 C CNN
-F 2 "" H 3450 2750 50  0001 C CNN
+F 2 "Connector_PinHeader_2.54mm:PinHeader_1x02_P2.54mm_Vertical" H 3450 2750 50  0001 C CNN
 F 3 "~" H 3450 2750 50  0001 C CNN
 	1    3450 2750

Commit message: Completes first cut of the schematic
Parts:
- BT?: value Battery_Cell -> 9V
Changed lines of the file:
@@
 AR Path="/61B8E1CE/61AE75FA" Ref="BT?"  Part="1"
 F 0 "BT?" H 3150 3100 50  0000 L CNN
-F 1 "Battery_Cell" V 3000 3000 50  0000 L CNN
+F 1 "9V" H 2950 3300 50  0000 L CNN
 F 2 "CoaxTester:BATT_CONN" V 3150 3210 50  0001 C CNN
 F 3 "~" V 3150 3210 50  0001 C CNN
