File: pcb/CoaxTester.sch (KiCad schematic (older format))
At the start: 14 parts

Commit message: Updates schematic based on some testing. Adds PDF for review
Other:
- note added: "HEAD"
- note added: "TAIL"
- moved on the sheet: C?, J?, R?, U?
