File: pcb/Head_Line_Driver.kicad_sch (KiCad schematic)
At the start: 9 parts

Commit message: Adds some controls and debounce.
Changed lines of the file:
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@@
     (stroke (width 0) (type default) (color 0 0 0 0))
   )
-  (wire (pts (xy 113.03 83.82) (xy 121.92 83.82))
+  (wire (pts (xy 107.315 83.82) (xy 121.92 83.82))
     (stroke (width 0) (type default) (color 0 0 0 0))
   )
@@
     (effects (font (size 1.27 1.27)) (justify left bottom))
   )
+  (global_label "5V" (shape input) (at 107.315 83.82 180) (fields_autoplaced)
+    (effects (font (size 1.27 1.27)) (justify right))
+    (property "Intersheet References" "${INTERSHEET_REFS}" (id 0) (at 102.6927 83.7406 0)
+      (effects (font (size 1.27 1.27)) (justify right) hide)
+    )
+  )
   (hierarchical_label "DATA_IN" (shape input) (at 342.9 162.56 0)
     (effects (font (size 1.27 1.27)) (justify left))
@@
     (effects (font (size 1.27 1.27)) (justify right))
   )
-  (hierarchical_label "5V" (shape input) (at 179.07 85.09 180)
-    (effects (font (size 1.27 1.27)) (justify right))
-  )

Commit message: Updates the schematic and fixes some symbols
Connections:
- net 5V: no longer U?.16 (VCC), U?.16 (VCC)
- new net 3V3: U?.16 (VCC), U?.16 (VCC)
Changed lines of the file:
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@@
     (stroke (width 0) (type default) (color 0 0 0 0))
   )
-  (wire (pts (xy 107.315 83.82) (xy 121.92 83.82))
+  (wire (pts (xy 113.665 83.82) (xy 121.92 83.82))
     (stroke (width 0) (type default) (color 0 0 0 0))
   )
@@
     (effects (font (size 1.27 1.27)) (justify right bottom))
   )
-  (label "5V" (at 285.75 139.7 0)
-    (effects (font (size 1.27 1.27)) (justify left bottom))
-  )
   (label "RCLK" (at 97.79 106.68 0)
     (effects (font (size 1.27 1.27)) (justify left bottom))
@@
     (effects (font (size 1.27 1.27)) (justify left bottom))
   )
-  (label "5V" (at 114.3 133.35 0)
-    (effects (font (size 1.27 1.27)) (justify left bottom))
-  )
   (label "5V" (at 106.68 101.6 0)
     (effects (font (size 1.27 1.27)) (justify left bottom))
@@
     (effects (font (size 1.27 1.27)) (justify right bottom))
   )
-  (label "5V" (at 113.03 83.82 0)
-    (effects (font (size 1.27 1.27)) (justify left bottom))
-  )
   (label "HD_VERT_CORE" (at 151.13 140.97 180)
     (effects (font (size 1.27 1.27)) (justify right bottom))
@@
     (effects (font (size 1.27 1.27)) (justify left bottom))
   )
+  (label "5V" (at 116.84 83.82 0)
+    (effects (font (size 1.27 1.27)) (justify left bottom))
+  )
   (label "RCLK" (at 88.9 153.67 0)
     (effects (font (size 1.27 1.27)) (justify left bottom))
@@
     (effects (font (size 1.27 1.27)) (justify left bottom))
   )
-  (label "5V" (at 285.75 69.85 0)
-    (effects (font (size 1.27 1.27)) (justify left bottom))
-  )
   (label "~{SH{slash}LD}" (at 269.24 106.68 0)
     (effects (font (size 1.27 1.27)) (justify left bottom))
@@
     (effects (font (size 1.27 1.27)) (justify left bottom))
   )
+  (label "5V" (at 116.84 133.35 0)
+    (effects (font (size 1.27 1.27)) (justify left bottom))
+  )
   (label "5V" (at 179.07 85.09 0)
     (effects (font (size 1.27 1.27)) (justify left bottom))
@@
     (effects (font (size 1.27 1.27)) (justify left bottom))
   )
-  (global_label "5V" (shape input) (at 107.315 83.82 180) (fields_autoplaced)
+  (global_label "3V3" (shape input) (at 285.75 139.7 180) (fields_autoplaced)
     (effects (font (size 1.27 1.27)) (justify right))
-    (property "Intersheet References" "${INTERSHEET_REFS}" (id 0) (at 102.6927 83.7406 0)
+    (property "Intersheet References" "${INTERSHEET_REFS}" (id 0) (at 279.9182 139.6206 0)
       (effects (font (size 1.27 1.27)) (justify right) hide)
     )
+  )
+  (global_label "5V" (shape input) (at 114.3 133.35 180) (fields_autoplaced)
+    (effects (font (size 1.27 1.27)) (justify right))
+    (property "Intersheet References" "${INTERSHEET_REFS}" (id 0) (at 109.6777 133.2706 0)
+      (effects (font (size 1.27 1.27)) (justify right) hide)
+    )
+  )
+  (global_label "5V" (shape input) (at 113.665 83.82 180) (fields_autoplaced)
+    (effects (font (size 1.27 1.27)) (justify right))
+    (property "Intersheet References" "${INTERSHEET_REFS}" (id 0) (at 109.0427 83.7406 0)
+      (effects (font (size 1.27 1.27)) (justify right) hide)
+    )
+  )
+  (global_label "3V3" (shape input) (at 285.75 69.85 180) (fields_autoplaced)
+    (effects (font (size 1.27 1.27)) (justify right))
+    (property "Intersheet References" "${INTERSHEET_REFS}" (id 0) (at 279.9182 69.7706 0)
+      (effects (font (size 1.27 1.27)) (justify right) hide)
+    )
