File: pcb/Head_Line_Driver.kicad_sch (KiCad schematic)
At the start: 9 parts

Commit message: Schematic complete
Parts:
- gave numbers to parts that had none: 9
Connections:
- net CLK_IN: no longer U801.11 (SRCLK), U802.11 (SRCLK)
- net 3V3 renamed +3.3V
- net 5V renamed +5V
- new net CLK_OUT: U801.11 (SRCLK), U802.11 (SRCLK)
Other:
- sheet CH01_02H ports: added none; removed 5V
- sheet CH03_04H ports: added none; removed 5V
- sheet CH05_06H ports: added none; removed 5V
- sheet CH07_08H ports: added none; removed 5V
- sheet CH09H ports: added none; removed 5V

Commit message: DRC pass
Connections:
- net +3.3V renamed Vdd
Changed lines of the file:
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@@
-    (stroke (width 0) (type default) (color 0 0 0 0))
-  )
-  (wire (pts (xy 290.83 73.66) (xy 290.83 72.39))
     (stroke (width 0) (type default) (color 0 0 0 0))
   )
@@
     (stroke (width 0) (type default) (color 0 0 0 0))
   )
+  (wire (pts (xy 290.83 69.85) (xy 290.83 73.66))
+    (stroke (width 0) (type default) (color 0 0 0 0))
+  )
   (wire (pts (xy 172.72 168.91) (xy 185.42 168.91))
     (stroke (width 0) (type default) (color 0 0 0 0))
@@
   )
   (wire (pts (xy 176.53 120.65) (xy 185.42 120.65))
+    (stroke (width 0) (type default) (color 0 0 0 0))
+  )
+  (wire (pts (xy 290.83 69.85) (xy 287.02 69.85))
     (stroke (width 0) (type default) (color 0 0 0 0))
   )
@@
     (effects (font (size 1.27 1.27)) (justify left bottom))
   )
+  (label "Vdd" (at 290.83 69.85 180)
+    (effects (font (size 1.27 1.27)) (justify right bottom))
+  )
   (label "HB_HORIZ_CORE" (at 151.13 99.06 180)
     (effects (font (size 1.27 1.27)) (justify right bottom))
@@
     (effects (font (size 1.27 1.27)) (justify right bottom))
   )
+  (label "Vdd" (at 290.83 142.24 0)
+    (effects (font (size 1.27 1.27)) (justify left bottom))
+  )
   (label "HD_HORIZ_SHIELD" (at 222.25 101.6 0)
     (effects (font (size 1.27 1.27)) (justify left bottom))
@@
   (label "~{Qh1}" (at 311.15 83.82 180)
     (effects (font (size 1.27 1.27)) (justify right bottom))
+  )
+  (hierarchical_label "Vdd" (shape input) (at 287.02 69.85 180)
+    (effects (font (size 1.27 1.27)) (justify right))
   )
   (hierarchical_label "DATA_IN" (shape input) (at 342.9 162.56 0)
@@
     )
     (property "Datasheet" "" (id 3) (at 290.83 195.58 0)
-      (effects (font (size 1.27 1.27)) hide)
-    )
-    (pin "1")
-  )
-  (symbol (lib_id "power:+3.3V") (at 290.83 72.39 0) (unit 1)
-    (in_bom yes) (on_board yes) (fields_autoplaced)
-    (property "Reference" "#PWR0811" (id 0) (at 290.83 76.2 0)
-      (effects (font (size 1.27 1.27)) hide)
-    )
-    (property "Value" "+3.3V" (id 1) (at 290.83 68.8142 0))
-    (property "Footprint" "" (id 2) (at 290.83 72.39 0)
-      (effects (font (size 1.27 1.27)) hide)
-    )
-    (property "Datasheet" "" (id 3) (at 290.83 72.39 0)
       (effects (font (size 1.27 1.27)) hide)
     )
@@
       (effects (font (size 1.27 1.27)) hide)
     )
-    (pin "1")
-  )
-  (symbol (lib_id "power:+3.3V") (at 290.83 142.24 0) (unit 1)
-    (in_bom yes) (on_board yes) (fields_autoplaced)
-    (property "Reference" "#PWR0813" (id 0) (at 290.83 146.05 0)
-      (effects (font (size 1.27 1.27)) hide)
-    )
-    (property "Value" "+3.3V" (id 1) (at 290.83 138.6642 0))
-    (property "Footprint" "" (id 2) (at 290.83 142.24 0)
-      (effects (font (size 1.27 1.27)) hide)
-    )
-    (property "Datasheet" "" (id 3) (at 290.83 142.24 0)
-      (effects (font (size 1.27 1.27)) hide)
-    )

Commit message: DRC OK
Parts:
- removed J801: CONF1, Jumper:SolderJumper-3_P1.3mm_Bridged12_RoundedPad1.0x1.5mm, symbol Connector:Conn_01x03_Male
- removed J802: CONF2, Jumper:SolderJumper-3_P1.3mm_Bridged12_RoundedPad1.0x1.5mm, symbol Connector:Conn_01x03_Male
- added J801, J802: Conn_01x03_Pin, Jumper:SolderJumper-3_P1.3mm_Bridged12_RoundedPad1.0x1.5mm, symbol Connector:Conn_01x03_Pin
Connections:
- net DATA_IN: now also J802.2 (Pin_2)
- net Qh: now also J801.1 (Pin_1), J801.2 (Pin_2)
- net ~{Qh1}: now also J801.3 (Pin_3)
- net ~{Qh2}: now also J802.3 (Pin_3)
- net at U804.9 (Q7): now also J802.1 (Pin_1)
