File: pcb/CH01_02H.kicad_sch (KiCad schematic)
At the start: 12 parts

Commit message: Schematic complete
Parts:
- gave numbers to parts that had none: 10
Connections:
- net 5V renamed +5V
Changed lines of the file:
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@@
     (stroke (width 0) (type default) (color 0 0 0 0))
   )
-  (wire (pts (xy 72.39 52.07) (xy 90.17 52.07))
+  (wire (pts (xy 82.55 52.07) (xy 90.17 52.07))
     (stroke (width 0) (type default) (color 0 0 0 0))
   )
@@
     (stroke (width 0) (type default) (color 0 0 0 0))
   )
-  (wire (pts (xy 109.22 44.45) (xy 100.33 44.45))
-    (stroke (width 0) (type default) (color 0 0 0 0))
-  )
-  (wire (pts (xy 73.66 121.92) (xy 91.44 121.92))
+  (wire (pts (xy 82.55 121.92) (xy 91.44 121.92))
     (stroke (width 0) (type default) (color 0 0 0 0))
   )
@@
     (stroke (width 0) (type default) (color 0 0 0 0))
   )
-  (wire (pts (xy 110.49 114.3) (xy 101.6 114.3))
-    (stroke (width 0) (type default) (color 0 0 0 0))
-  )
   (wire (pts (xy 110.49 116.84) (xy 110.49 114.3))
     (stroke (width 0) (type default) (color 0 0 0 0))
-  )
-  (label "5V" (at 101.6 114.3 0)
-    (effects (font (size 1.27 1.27)) (justify left bottom))
-  )
-  (label "5V" (at 100.33 44.45 0)
-    (effects (font (size 1.27 1.27)) (justify left bottom))
   )
   (hierarchical_label "HORIZ_SHIELD" (shape input) (at 149.86 81.28 0)
@@
     (effects (font (size 1.27 1.27)) (justify left))
   )
-  (hierarchical_label "HORIZ_CORE" (shape input) (at 72.39 52.07 180)
+  (hierarchical_label "HORIZ_CORE" (shape input) (at 82.55 52.07 180)
     (effects (font (size 1.27 1.27)) (justify right))
   )
-  (hierarchical_label "5V" (shape input) (at 100.33 44.45 180)
+  (hierarchical_label "VERT_CORE" (shape input) (at 82.55 121.92 180)
     (effects (font (size 1.27 1.27)) (justify right))
   )
-  (hierarchical_label "VERT_CORE" (shape input) (at 73.66 121.92 180)
-    (effects (font (size 1.27 1.27)) (justify right))
-  )
   (symbol (lib_id "Device:R") (at 116.84 87.63 0) (unit 1)
     (in_bom yes) (on_board yes)
-    (property "Reference" "R?" (id 0) (at 118.618 86.4616 0)
+    (property "Reference" "R204" (id 0) (at 118.618 86.4616 0)
       (effects (font (size 1.27 1.27)) (justify left))
     )
@@
   (symbol (lib_id "Device:R") (at 118.11 140.97 0) (unit 1)
     (in_bom yes) (on_board yes)
-    (property "Reference" "R?" (id 0) (at 119.888 139.8016 0)
+    (property "Reference" "R205" (id 0) (at 119.888 139.8016 0)
       (effects (font (size 1.27 1.27)) (justify left))
     )
@@
   (symbol (lib_id "power:GND") (at 118.11 157.48 0) (unit 1)
     (in_bom yes) (on_board yes)
-    (property "Reference" "#PWR?" (id 0) (at 118.11 163.83 0)
+    (property "Reference" "#PWR0204" (id 0) (at 118.11 163.83 0)
       (effects (font (size 1.27 1.27)) hide)
     )
@@
   (symbol (lib_id "Device:R") (at 118.11 152.4 0) (unit 1)
     (in_bom yes) (on_board yes)
-    (property "Reference" "R?" (id 0) (at 119.888 151.2316 0)
+    (property "Reference" "R206" (id 0) (at 119.888 151.2316 0)
       (effects (font (size 1.27 1.27)) (justify left))
     )
@@
   (symbol (lib_id "Connector:Conn_Coaxial") (at 116.84 59.69 0) (unit 1)
     (in_bom yes) (on_board yes)
-    (property "Reference" "J?" (id 0) (at 119.38 60.325 0)
+    (property "Reference" "J201" (id 0) (at 119.38 60.325 0)
       (effects (font (size 1.27 1.27)) (justify left))
     )
@@
   (symbol (lib_id "Device:R") (at 93.98 52.07 270) (unit 1)
     (in_bom yes) (on_board yes)
-    (property "Reference" "R?" (id 0) (at 93.98 46.8122 90))
+    (property "Reference" "R201" (id 0) (at 93.98 46.8122 90))
     (property "Value" "500Ω" (id 1) (at 93.98 49.1236 90))
     (property "Footprint" "Resistor_SMD:R_0805_2012Metric" (id 2) (at 93.98 50.292 90)
@@
   (symbol (lib_id "Device:R") (at 116.84 74.93 0) (unit 1)
     (in_bom yes) (on_board yes)
-    (property "Reference" "R?" (id 0) (at 118.618 73.7616 0)
+    (property "Reference" "R203" (id 0) (at 118.618 73.7616 0)
       (effects (font (size 1.27 1.27)) (justify left))
     )
@@
   (symbol (lib_id "power:GND") (at 116.84 92.71 0) (unit 1)
     (in_bom yes) (on_board yes)
-    (property "Reference" "#PWR?" (id 0) (at 116.84 99.06 0)
+    (property "Reference" "#PWR0203" (id 0) (at 116.84 99.06 0)
       (effects (font (size 1.27 1.27)) hide)
     )
@@
   (symbol (lib_id "Connector:Conn_Coaxial") (at 118.11 130.81 0) (unit 1)
     (in_bom yes) (on_board yes)
-    (property "Reference" "J?" (id 0) (at 120.65 131.445 0)
+    (property "Reference" "J202" (id 0) (at 120.65 131.445 0)
       (effects (font (size 1.27 1.27)) (justify left))
     )
@@
   (symbol (lib_id "Device:R") (at 95.25 121.92 270) (unit 1)
     (in_bom yes) (on_board yes)
-    (property "Reference" "R?" (id 0) (at 95.25 116.6622 90))
+    (property "Reference" "R202" (id 0) (at 95.25 116.6622 90))
     (property "Value" "500Ω" (id 1) (at 95.25 118.9736 90))
     (property "Footprint" "Resistor_SMD:R_0805_2012Metric" (id 2) (at 95.25 120.142 90)
@@
   (symbol (lib_id "power:GND") (at 146.05 182.88 0) (unit 1)
     (in_bom yes) (on_board yes)
-    (property "Reference" "#PWR?" (id 0) (at 146.05 189.23 0)
+    (property "Reference" "#PWR0206" (id 0) (at 146.05 189.23 0)
       (effects (font (size 1.27 1.27)) hide)
     )
@@
     (pin "1")
   )
+  (symbol (lib_id "power:+5V") (at 109.22 44.45 0) (unit 1)
+    (in_bom yes) (on_board yes) (fields_autoplaced)
+    (property "Reference" "#PWR0201" (id 0) (at 109.22 48.26 0)
+      (effects (font (size 1.27 1.27)) hide)
+    )
+    (property "Value" "+5V" (id 1) (at 109.22 40.8742 0))
+    (property "Footprint" "" (id 2) (at 109.22 44.45 0)
+      (effects (font (size 1.27 1.27)) hide)
+    )
+    (property "Datasheet" "" (id 3) (at 109.22 44.45 0)
+      (effects (font (size 1.27 1.27)) hide)
+    )
+    (pin "1")
+  )
   (symbol (lib_id "Transistor_BJT:BC847BPN") (at 106.68 52.07 0) (unit 1)
     (in_bom yes) (on_board yes) (fields_autoplaced)
-    (property "Reference" "Q?" (id 0) (at 111.5314 51.1615 0)
+    (property "Reference" "Q201" (id 0) (at 111.5314 51.1615 0)
       (effects (font (size 1.27 1.27)) (justify left))
     )
@@
     (pin "2")
     (pin "6")
-  )
-  (symbol (lib_id "Transistor_BJT:BC847BPN") (at 107.95 121.92 0) (unit 2)
-    (in_bom yes) (on_board yes) (fields_autoplaced)
-    (property "Reference" "Q?" (id 0) (at 112.8014 121.0115 0)
-      (effects (font (size 1.27 1.27)) (justify left))
-    )
-    (property "Value" "BC847BPN" (id 1) (at 112.8014 123.7866 0)
-      (effects (font (size 1.27 1.27)) (justify left))
-    )
-    (property "Footprint" "Package_TO_SOT_SMD:SOT-363_SC-70-6" (id 2) (at 113.03 119.38 0)
-      (effects (font (size 1.27 1.27)) hide)
-    )
-    (property "Datasheet" "https://assets.nexperia.com/documents/data-sheet/BC847BPN.pdf" (id 3) (at 107.95 121.92 0)
-      (effects (font (size 1.27 1.27)) hide)
-    )
     (pin "3")
     (pin "4")
     (pin "5")
   )
+  (symbol (lib_id "power:+5V") (at 110.49 114.3 0) (unit 1)
+    (in_bom yes) (on_board yes) (fields_autoplaced)
+    (property "Reference" "#PWR0202" (id 0) (at 110.49 118.11 0)
+      (effects (font (size 1.27 1.27)) hide)
+    )
+    (property "Value" "+5V" (id 1) (at 110.49 110.7242 0))
+    (property "Footprint" "" (id 2) (at 110.49 114.3 0)
+      (effects (font (size 1.27 1.27)) hide)
+    )
+    (property "Datasheet" "" (id 3) (at 110.49 114.3 0)
+      (effects (font (size 1.27 1.27)) hide)
+    )
+    (pin "1")
+  )
+  (symbol (lib_id "Transistor_BJT:BC847BPN") (at 107.95 121.92 0) (unit 2)
+    (in_bom yes) (on_board yes) (fields_autoplaced)
+    (property "Reference" "Q201" (id 0) (at 112.8014 121.0115 0)
+      (effects (font (size 1.27 1.27)) (justify left))
+    )
+    (property "Value" "BC847BPN" (id 1) (at 112.8014 123.7866 0)
+      (effects (font (size 1.27 1.27)) (justify left))
+    )
+    (property "Footprint" "Package_TO_SOT_SMD:SOT-363_SC-70-6" (id 2) (at 113.03 119.38 0)
+      (effects (font (size 1.27 1.27)) hide)
+    )
+    (property "Datasheet" "https://assets.nexperia.com/documents/data-sheet/BC847BPN.pdf" (id 3) (at 107.95 121.92 0)
+      (effects (font (size 1.27 1.27)) hide)
+    )
+    (pin "1")
+    (pin "2")
+    (pin "6")
+    (pin "3")
+    (pin "4")
+    (pin "5")
+  )
   (symbol (lib_id "CoaxTester:SMDB03C") (at 146.05 102.87 0) (unit 1)
     (in_bom yes) (on_board yes) (fields_autoplaced)
-    (property "Reference" "D?" (id 0) (at 149.5552 102.0353 0)
+    (property "Reference" "D201" (id 0) (at 149.5552 102.0353 0)
       (effects (font (size 1.27 1.27)) (justify left))
     )
@@
     (pin "1")
     (pin "8")
+    (pin "2")
+    (pin "7")
+    (pin "3")
+    (pin "6")
+    (pin "4")
+    (pin "5")
   )
   (symbol (lib_id "power:GND") (at 146.05 118.11 0) (unit 1)
     (in_bom yes) (on_board yes)
-    (property "Reference" "#PWR?" (id 0) (at 146.05 124.46 0)
+    (property "Reference" "#PWR0205" (id 0) (at 146.05 124.46 0)
       (effects (font (size 1.27 1.27)) hide)
     )
@@
   (symbol (lib_id "CoaxTester:SMDB03C") (at 146.05 166.37 0) (unit 2)
     (in_bom yes) (on_board yes) (fields_autoplaced)
-    (property "Reference" "D?" (id 0) (at 149.5552 165.5353 0)
+    (property "Reference" "D201" (id 0) (at 149.5552 165.5353 0)
       (effects (font (size 1.27 1.27)) (justify left))
     )
@@
       (effects (font (size 1.27 1.27)) hide)
     )
+    (pin "1")
+    (pin "8")
     (pin "2")
     (pin "7")
+    (pin "3")
+    (pin "6")
+    (pin "4")
+    (pin "5")
   )
 )
