File: pcb/CH05_06H.kicad_sch (KiCad schematic)
At the start: 12 parts

Commit message: Schematic complete
Parts:
- gave numbers to parts that had none: 10
Connections:
- net 5V renamed +5V
Changed lines of the file:
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@@
-    (stroke (width 0) (type default) (color 0 0 0 0))
-  )
-  (wire (pts (xy 109.22 44.45) (xy 104.14 44.45))
     (stroke (width 0) (type default) (color 0 0 0 0))
   )
@@
     (stroke (width 0) (type default) (color 0 0 0 0))
   )
-  (wire (pts (xy 109.22 110.49) (xy 105.41 110.49))
-    (stroke (width 0) (type default) (color 0 0 0 0))
-  )
   (wire (pts (xy 109.22 113.03) (xy 109.22 110.49))
     (stroke (width 0) (type default) (color 0 0 0 0))
@@
   (wire (pts (xy 149.86 142.24) (xy 149.86 152.4))
     (stroke (width 0) (type default) (color 0 0 0 0))
-  )
-  (label "5V" (at 105.41 110.49 0)
-    (effects (font (size 1.27 1.27)) (justify left bottom))
-  )
-  (label "5V" (at 105.41 44.45 0)
-    (effects (font (size 1.27 1.27)) (justify left bottom))
   )
   (hierarchical_label "HORIZ_SHIELD" (shape input) (at 153.67 76.2 0)
@@
     (effects (font (size 1.27 1.27)) (justify right))
   )
-  (hierarchical_label "5V" (shape input) (at 104.14 44.45 180)
-    (effects (font (size 1.27 1.27)) (justify right))
-  )
   (symbol (lib_id "Device:R") (at 96.52 52.07 270) (unit 1)
     (in_bom yes) (on_board yes)
-    (property "Reference" "R?" (id 0) (at 96.52 46.8122 90))
+    (property "Reference" "R402" (id 0) (at 96.52 46.8122 90))
     (property "Value" "500Ω" (id 1) (at 96.52 49.1236 90))
     (property "Footprint" "Resistor_SMD:R_0805_2012Metric" (id 2) (at 96.52 50.292 90)
@@
   (symbol (lib_id "Device:R") (at 115.57 69.85 0) (unit 1)
     (in_bom yes) (on_board yes)
-    (property "Reference" "R?" (id 0) (at 117.348 68.6816 0)
+    (property "Reference" "R403" (id 0) (at 117.348 68.6816 0)
       (effects (font (size 1.27 1.27)) (justify left))
     )
@@
   (symbol (lib_id "power:GND") (at 115.57 87.63 0) (unit 1)
     (in_bom yes) (on_board yes)
-    (property "Reference" "#PWR?" (id 0) (at 115.57 93.98 0)
+    (property "Reference" "#PWR0403" (id 0) (at 115.57 93.98 0)
       (effects (font (size 1.27 1.27)) hide)
     )
@@
   (symbol (lib_id "Device:R") (at 115.57 82.55 0) (unit 1)
     (in_bom yes) (on_board yes)
-    (property "Reference" "R?" (id 0) (at 117.348 81.3816 0)
+    (property "Reference" "R404" (id 0) (at 117.348 81.3816 0)
       (effects (font (size 1.27 1.27)) (justify left))
     )
@@
   (symbol (lib_id "Device:R") (at 115.57 135.89 0) (unit 1)
     (in_bom yes) (on_board yes)
-    (property "Reference" "R?" (id 0) (at 117.348 134.7216 0)
+    (property "Reference" "R405" (id 0) (at 117.348 134.7216 0)
       (effects (font (size 1.27 1.27)) (justify left))
     )
@@
   (symbol (lib_id "power:GND") (at 115.57 154.94 0) (unit 1)
     (in_bom yes) (on_board yes)
-    (property "Reference" "#PWR?" (id 0) (at 115.57 161.29 0)
+    (property "Reference" "#PWR0404" (id 0) (at 115.57 161.29 0)
       (effects (font (size 1.27 1.27)) hide)
     )
@@
   (symbol (lib_id "Device:R") (at 115.57 148.59 0) (unit 1)
     (in_bom yes) (on_board yes)
-    (property "Reference" "R?" (id 0) (at 117.348 147.4216 0)
+    (property "Reference" "R406" (id 0) (at 117.348 147.4216 0)
       (effects (font (size 1.27 1.27)) (justify left))
     )
@@
   (symbol (lib_id "Connector:Conn_Coaxial") (at 115.57 59.69 0) (unit 1)
     (in_bom yes) (on_board yes)
-    (property "Reference" "J?" (id 0) (at 118.11 60.325 0)
+    (property "Reference" "J401" (id 0) (at 118.11 60.325 0)
       (effects (font (size 1.27 1.27)) (justify left))
     )
@@
   (symbol (lib_id "Connector:Conn_Coaxial") (at 115.57 125.73 0) (unit 1)
     (in_bom yes) (on_board yes)
-    (property "Reference" "J?" (id 0) (at 118.11 126.365 0)
+    (property "Reference" "J402" (id 0) (at 118.11 126.365 0)
       (effects (font (size 1.27 1.27)) (justify left))
     )
@@
   (symbol (lib_id "Device:R") (at 93.98 118.11 270) (unit 1)
     (in_bom yes) (on_board yes)
-    (property "Reference" "R?" (id 0) (at 93.98 112.8522 90))
+    (property "Reference" "R401" (id 0) (at 93.98 112.8522 90))
     (property "Value" "500Ω" (id 1) (at 93.98 115.1636 90))
     (property "Footprint" "Resistor_SMD:R_0805_2012Metric" (id 2) (at 93.98 116.332 90)
@@
   (symbol (lib_id "Transistor_BJT:BC847BPN") (at 106.68 118.11 0) (unit 2)
     (in_bom yes) (on_board yes) (fields_autoplaced)
-    (property "Reference" "Q?" (id 0) (at 111.5314 117.2015 0)
+    (property "Reference" "Q401" (id 0) (at 111.5314 117.2015 0)
       (effects (font (size 1.27 1.27)) (justify left))
     )
@@
       (effects (font (size 1.27 1.27)) hide)
     )
+    (pin "1")
+    (pin "2")
+    (pin "6")
     (pin "3")
     (pin "4")
@@
   (symbol (lib_id "power:GND") (at 149.86 179.07 0) (unit 1)
     (in_bom yes) (on_board yes)
-    (property "Reference" "#PWR?" (id 0) (at 149.86 185.42 0)
+    (property "Reference" "#PWR0406" (id 0) (at 149.86 185.42 0)
       (effects (font (size 1.27 1.27)) hide)
     )
@@
     (pin "1")
   )
-  (symbol (lib_id "CoaxTester:SMDB03C") (at 149.86 91.44 0) (unit 1)
-    (in_bom yes) (on_board yes) (fields_autoplaced)
-    (property "Reference" "D?" (id 0) (at 153.3652 90.6053 0)
+  (symbol (lib_id "power:+5V") (at 109.22 44.45 0) (unit 1)
+    (in_bom yes) (on_board yes) (fields_autoplaced)
+    (property "Reference" "#PWR0401" (id 0) (at 109.22 48.26 0)
+      (effects (font (size 1.27 1.27)) hide)
+    )
+    (property "Value" "+5V" (id 1) (at 109.22 40.8742 0))
+    (property "Footprint" "" (id 2) (at 109.22 44.45 0)
+      (effects (font (size 1.27 1.27)) hide)
+    )
+    (property "Datasheet" "" (id 3) (at 109.22 44.45 0)
+      (effects (font (size 1.27 1.27)) hide)
+    )
+    (pin "1")
+  )
+  (symbol (lib_id "power:+5V") (at 109.22 110.49 0) (unit 1)
+    (in_bom yes) (on_board yes) (fields_autoplaced)
+    (property "Reference" "#PWR0402" (id 0) (at 109.22 114.3 0)
+      (effects (font (size 1.27 1.27)) hide)
+    )
+    (property "Value" "+5V" (id 1) (at 109.22 106.9142 0))
+    (property "Footprint" "" (id 2) (at 109.22 110.49 0)
+      (effects (font (size 1.27 1.27)) hide)
+    )
+    (property "Datasheet" "" (id 3) (at 109.22 110.49 0)
+      (effects (font (size 1.27 1.27)) hide)
+    )
+    (pin "1")
+  )
+  (symbol (lib_name "SMDB03C_1") (lib_id "CoaxTester:SMDB03C") (at 149.86 91.44 0) (unit 1)
+    (in_bom yes) (on_board yes) (fields_autoplaced)
+    (property "Reference" "D401" (id 0) (at 153.3652 90.6053 0)
       (effects (font (size 1.27 1.27)) (justify left))
     )
@@
     (pin "1")
     (pin "8")
+    (pin "2")
+    (pin "7")
+    (pin "3")
+    (pin "6")
+    (pin "4")
+    (pin "5")
   )
   (symbol (lib_id "CoaxTester:SMDB03C") (at 149.86 163.83 0) (unit 2)
     (in_bom yes) (on_board yes) (fields_autoplaced)
-    (property "Reference" "D?" (id 0) (at 153.3652 162.9953 0)
+    (property "Reference" "D401" (id 0) (at 153.3652 162.9953 0)
       (effects (font (size 1.27 1.27)) (justify left))
     )
@@
       (effects (font (size 1.27 1.27)) hide)
     )
+    (pin "1")
+    (pin "8")
     (pin "2")
     (pin "7")
+    (pin "3")
+    (pin "6")
+    (pin "4")
+    (pin "5")
   )
   (symbol (lib_id "Transistor_BJT:BC847BPN") (at 106.68 52.07 0) (unit 1)
     (in_bom yes) (on_board yes) (fields_autoplaced)
-    (property "Reference" "Q?" (id 0) (at 111.5314 51.1615 0)
+    (property "Reference" "Q401" (id 0) (at 111.5314 51.1615 0)
       (effects (font (size 1.27 1.27)) (justify left))
     )
@@
     (pin "2")
     (pin "6")
+    (pin "3")
+    (pin "4")
+    (pin "5")
   )
   (symbol (lib_id "power:GND") (at 149.86 106.68 0) (unit 1)
     (in_bom yes) (on_board yes)
-    (property "Reference" "#PWR?" (id 0) (at 149.86 113.03 0)
-      (effects (font (size 1.27 1.27)) hide)
-    )
+    (property "Reference" "#PWR0405" (id 0) (at 149.86 113.03 0)
+      (effects (font (size 1.27 1.27)) hide)
+    )
