File: pcb/CH07_08H.kicad_sch (KiCad schematic)
At the start: 12 parts

Commit message: Schematic complete
Parts:
- gave numbers to parts that had none: 10
Connections:
- net 5V renamed +5V
Changed lines of the file:
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@@
-    (stroke (width 0) (type default) (color 0 0 0 0))
-  )
-  (wire (pts (xy 109.22 44.45) (xy 105.41 44.45))
     (stroke (width 0) (type default) (color 0 0 0 0))
   )
@@
     (stroke (width 0) (type default) (color 0 0 0 0))
   )
-  (wire (pts (xy 109.22 106.68) (xy 105.41 106.68))
-    (stroke (width 0) (type default) (color 0 0 0 0))
-  )
   (wire (pts (xy 88.9 52.07) (xy 90.17 52.07))
     (stroke (width 0) (type default) (color 0 0 0 0))
@@
   (wire (pts (xy 115.57 64.77) (xy 115.57 66.04))
     (stroke (width 0) (type default) (color 0 0 0 0))
-  )
-  (label "5V" (at 105.41 106.68 0)
-    (effects (font (size 1.27 1.27)) (justify left bottom))
-  )
-  (label "5V" (at 105.41 44.45 0)
-    (effects (font (size 1.27 1.27)) (justify left bottom))
   )
   (hierarchical_label "HORIZ_CORE" (shape input) (at 88.9 52.07 180)
@@
     (effects (font (size 1.27 1.27)) (justify left))
   )
-  (hierarchical_label "5V" (shape input) (at 105.41 44.45 180)
-    (effects (font (size 1.27 1.27)) (justify right))
-  )
   (symbol (lib_id "Device:R") (at 115.57 69.85 0) (unit 1)
     (in_bom yes) (on_board yes)
-    (property "Reference" "R?" (id 0) (at 117.348 68.6816 0)
+    (property "Reference" "R505" (id 0) (at 117.348 68.6816 0)
       (effects (font (size 1.27 1.27)) (justify left))
     )
@@
   (symbol (lib_id "power:GND") (at 115.57 86.36 0) (unit 1)
     (in_bom yes) (on_board yes)
-    (property "Reference" "#PWR?" (id 0) (at 115.57 92.71 0)
+    (property "Reference" "#PWR0504" (id 0) (at 115.57 92.71 0)
       (effects (font (size 1.27 1.27)) hide)
     )
@@
   (symbol (lib_id "Device:R") (at 115.57 80.01 0) (unit 1)
     (in_bom yes) (on_board yes)
-    (property "Reference" "R?" (id 0) (at 117.348 78.8416 0)
+    (property "Reference" "R506" (id 0) (at 117.348 78.8416 0)
       (effects (font (size 1.27 1.27)) (justify left))
     )
@@
   (symbol (lib_id "Device:R") (at 114.3 132.08 0) (unit 1)
     (in_bom yes) (on_board yes)
-    (property "Reference" "R?" (id 0) (at 116.078 130.9116 0)
+    (property "Reference" "R503" (id 0) (at 116.078 130.9116 0)
       (effects (font (size 1.27 1.27)) (justify left))
     )
@@
   (symbol (lib_id "power:GND") (at 114.3 149.86 0) (unit 1)
     (in_bom yes) (on_board yes)
-    (property "Reference" "#PWR?" (id 0) (at 114.3 156.21 0)
+    (property "Reference" "#PWR0503" (id 0) (at 114.3 156.21 0)
       (effects (font (size 1.27 1.27)) hide)
     )
@@
   (symbol (lib_id "Device:R") (at 114.3 143.51 0) (unit 1)
     (in_bom yes) (on_board yes)
-    (property "Reference" "R?" (id 0) (at 116.078 142.3416 0)
+    (property "Reference" "R504" (id 0) (at 116.078 142.3416 0)
       (effects (font (size 1.27 1.27)) (justify left))
     )
@@
   (symbol (lib_id "Connector:Conn_Coaxial") (at 115.57 59.69 0) (unit 1)
     (in_bom yes) (on_board yes)
-    (property "Reference" "J?" (id 0) (at 118.11 60.325 0)
+    (property "Reference" "J502" (id 0) (at 118.11 60.325 0)
       (effects (font (size 1.27 1.27)) (justify left))
     )
@@
   (symbol (lib_id "Device:R") (at 93.98 52.07 270) (unit 1)
     (in_bom yes) (on_board yes)
-    (property "Reference" "R?" (id 0) (at 93.98 46.8122 90))
+    (property "Reference" "R501" (id 0) (at 93.98 46.8122 90))
     (property "Value" "500Ω" (id 1) (at 93.98 49.1236 90))
     (property "Footprint" "Resistor_SMD:R_0805_2012Metric" (id 2) (at 93.98 50.292 90)
@@
   (symbol (lib_id "Connector:Conn_Coaxial") (at 114.3 121.92 0) (unit 1)
     (in_bom yes) (on_board yes)
-    (property "Reference" "J?" (id 0) (at 116.84 122.555 0)
+    (property "Reference" "J501" (id 0) (at 116.84 122.555 0)
       (effects (font (size 1.27 1.27)) (justify left))
     )
@@
   (symbol (lib_id "Device:R") (at 93.98 114.3 270) (unit 1)
     (in_bom yes) (on_board yes)
-    (property "Reference" "R?" (id 0) (at 93.98 109.0422 90))
+    (property "Reference" "R502" (id 0) (at 93.98 109.0422 90))
     (property "Value" "500Ω" (id 1) (at 93.98 111.3536 90))
     (property "Footprint" "Resistor_SMD:R_0805_2012Metric" (id 2) (at 93.98 112.522 90)
@@
     (pin "2")
   )
+  (symbol (lib_id "power:+5V") (at 109.22 44.45 0) (unit 1)
+    (in_bom yes) (on_board yes) (fields_autoplaced)
+    (property "Reference" "#PWR0501" (id 0) (at 109.22 48.26 0)
+      (effects (font (size 1.27 1.27)) hide)
+    )
+    (property "Value" "+5V" (id 1) (at 109.22 40.8742 0))
+    (property "Footprint" "" (id 2) (at 109.22 44.45 0)
+      (effects (font (size 1.27 1.27)) hide)
+    )
+    (property "Datasheet" "" (id 3) (at 109.22 44.45 0)
+      (effects (font (size 1.27 1.27)) hide)
+    )
+    (pin "1")
+  )
   (symbol (lib_id "power:GND") (at 158.75 168.91 0) (unit 1)
     (in_bom yes) (on_board yes)
-    (property "Reference" "#PWR?" (id 0) (at 158.75 175.26 0)
+    (property "Reference" "#PWR0506" (id 0) (at 158.75 175.26 0)
       (effects (font (size 1.27 1.27)) hide)
     )
@@
   (symbol (lib_id "CoaxTester:SMDB03C") (at 158.75 153.67 0) (unit 4)
     (in_bom yes) (on_board yes) (fields_autoplaced)
-    (property "Reference" "D?" (id 0) (at 162.2552 152.8353 0)
+    (property "Reference" "D501" (id 0) (at 162.2552 152.8353 0)
       (effects (font (size 1.27 1.27)) (justify left))
     )
@@
       (effects (font (size 1.27 1.27)) hide)
     )
+    (pin "1")
+    (pin "8")
+    (pin "2")
+    (pin "7")
+    (pin "3")
+    (pin "6")
     (pin "4")
     (pin "5")
@@
   (symbol (lib_id "Transistor_BJT:BC847BPN") (at 106.68 114.3 0) (unit 2)
     (in_bom yes) (on_board yes) (fields_autoplaced)
-    (property "Reference" "Q?" (id 0) (at 111.5314 113.3915 0)
+    (property "Reference" "Q501" (id 0) (at 111.5314 113.3915 0)
       (effects (font (size 1.27 1.27)) (justify left))
     )
@@
       (effects (font (size 1.27 1.27)) hide)
     )
+    (pin "1")
+    (pin "2")
+    (pin "6")
     (pin "3")
     (pin "4")
     (pin "5")
   )
+  (symbol (lib_id "power:+5V") (at 109.22 106.68 0) (unit 1)
+    (in_bom yes) (on_board yes) (fields_autoplaced)
+    (property "Reference" "#PWR0502" (id 0) (at 109.22 110.49 0)
+      (effects (font (size 1.27 1.27)) hide)
+    )
+    (property "Value" "+5V" (id 1) (at 109.22 103.1042 0))
+    (property "Footprint" "" (id 2) (at 109.22 106.68 0)
+      (effects (font (size 1.27 1.27)) hide)
+    )
+    (property "Datasheet" "" (id 3) (at 109.22 106.68 0)
+      (effects (font (size 1.27 1.27)) hide)
+    )
+    (pin "1")
+  )
   (symbol (lib_id "power:GND") (at 158.75 105.41 0) (unit 1)
     (in_bom yes) (on_board yes)
-    (property "Reference" "#PWR?" (id 0) (at 158.75 111.76 0)
+    (property "Reference" "#PWR0505" (id 0) (at 158.75 111.76 0)
       (effects (font (size 1.27 1.27)) hide)
     )
@@
   (symbol (lib_id "Transistor_BJT:BC847BPN") (at 106.68 52.07 0) (unit 1)
     (in_bom yes) (on_board yes) (fields_autoplaced)
-    (property "Reference" "Q?" (id 0) (at 111.5314 51.1615 0)
+    (property "Reference" "Q501" (id 0) (at 111.5314 51.1615 0)
       (effects (font (size 1.27 1.27)) (justify left))
     )
@@
     (pin "2")
     (pin "6")
-  )
-  (symbol (lib_id "CoaxTester:SMDB03C") (at 158.75 90.17 0) (unit 3)
-    (in_bom yes) (on_board yes) (fields_autoplaced)
-    (property "Reference" "D?" (id 0) (at 162.2552 89.3353 0)
+    (pin "3")
+    (pin "4")
+    (pin "5")
+  )
+  (symbol (lib_name "SMDB03C_1") (lib_id "CoaxTester:SMDB03C") (at 158.75 90.17 0) (unit 3)
+    (in_bom yes) (on_board yes) (fields_autoplaced)
+    (property "Reference" "D501" (id 0) (at 162.2552 89.3353 0)
       (effects (font (size 1.27 1.27)) (justify left))
     )
@@
       (effects (font (size 1.27 1.27)) hide)
     )
+    (pin "1")
+    (pin "8")
+    (pin "2")
+    (pin "7")
     (pin "3")
     (pin "6")
+    (pin "4")
+    (pin "5")
   )
 )

Commit message: DRC OK
Parts:
- renumbered D501 to D401
