File: pcb/TailPower.kicad_sch (KiCad schematic)
At the start: 5 parts

Commit message: Adds line protection
Connections:
- net GND2: now also U?.1 (GND)
Changed lines of the file:
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@@
+    (stroke (width 0) (type default) (color 0 0 0 0))
+  )
+  (wire (pts (xy 139.7 60.96) (xy 139.7 63.5))
     (stroke (width 0) (type default) (color 0 0 0 0))
   )
@@
       (effects (font (size 1.27 1.27)) hide)
     )
+    (pin "1")
+  )
+  (symbol (lib_id "power:GND2") (at 139.7 63.5 0) (unit 1)
+    (in_bom yes) (on_board yes)
+    (property "Reference" "#PWR?" (id 0) (at 139.7 69.85 0)
+      (effects (font (size 1.27 1.27)) hide)
+    )
+    (property "Value" "GND2" (id 1) (at 139.827 67.8942 0))
+    (property "Footprint" "" (id 2) (at 139.7 63.5 0)
+      (effects (font (size 1.27 1.27)) hide)
+    )
+    (property "Datasheet" "" (id 3) (at 139.7 63.5 0)
+      (effects (font (size 1.27 1.27)) hide)
+    )

Commit message: Adds current control for the display adapter back light
Changed lines of the file:
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@@
   (junction (at 128.27 69.85) (diameter 0) (color 0 0 0 0)
   )
+  (junction (at 123.444 69.85) (diameter 0) (color 0 0 0 0)
+  )
   (junction (at 125.73 69.85) (diameter 0) (color 0 0 0 0)
   )
   (junction (at 151.13 53.34) (diameter 0) (color 0 0 0 0)
   )
+  (junction (at 162.179 53.34) (diameter 0) (color 0 0 0 0)
+  )
   (junction (at 128.27 53.34) (diameter 0) (color 0 0 0 0)
   )
@@
     (stroke (width 0) (type default) (color 0 0 0 0))
   )
+  (wire (pts (xy 162.179 53.34) (xy 163.83 53.34))
+    (stroke (width 0) (type default) (color 0 0 0 0))
+  )
   (wire (pts (xy 151.13 53.34) (xy 147.32 53.34))
     (stroke (width 0) (type default) (color 0 0 0 0))
   )
-  (wire (pts (xy 106.68 69.85) (xy 125.73 69.85))
+  (wire (pts (xy 106.68 69.85) (xy 123.444 69.85))
     (stroke (width 0) (type default) (color 0 0 0 0))
   )
@@
     (stroke (width 0) (type default) (color 0 0 0 0))
   )
-  (wire (pts (xy 151.13 53.34) (xy 163.83 53.34))
+  (wire (pts (xy 123.444 69.85) (xy 125.73 69.85))
+    (stroke (width 0) (type default) (color 0 0 0 0))
+  )
+  (wire (pts (xy 151.13 53.34) (xy 162.179 53.34))
     (stroke (width 0) (type default) (color 0 0 0 0))
   )
@@
       (effects (font (size 1.27 1.27)) hide)
     )
+    (pin "1")
+  )
+  (symbol (lib_id "power:PWR_FLAG") (at 162.179 53.34 0) (unit 1)
+    (in_bom yes) (on_board yes) (fields_autoplaced)
+    (property "Reference" "#FLG?" (id 0) (at 162.179 51.435 0)
+      (effects (font (size 1.27 1.27)) hide)
+    )
+    (property "Value" "PWR_FLAG" (id 1) (at 162.179 49.7642 0))
+    (property "Footprint" "" (id 2) (at 162.179 53.34 0)
+      (effects (font (size 1.27 1.27)) hide)
+    )
+    (property "Datasheet" "~" (id 3) (at 162.179 53.34 0)
+      (effects (font (size 1.27 1.27)) hide)
+    )
+    (pin "1")
+  )
+  (symbol (lib_id "power:PWR_FLAG") (at 123.444 69.85 0) (unit 1)
+    (in_bom yes) (on_board yes) (fields_autoplaced)
+    (property "Reference" "#FLG?" (id 0) (at 123.444 67.945 0)
+      (effects (font (size 1.27 1.27)) hide)
+    )
+    (property "Value" "PWR_FLAG" (id 1) (at 123.444 66.2742 0))
+    (property "Footprint" "" (id 2) (at 123.444 69.85 0)
+      (effects (font (size 1.27 1.27)) hide)
+    )
+    (property "Datasheet" "~" (id 3) (at 123.444 69.85 0)
+      (effects (font (size 1.27 1.27)) hide)
+    )

Commit message: Schematic complete
Parts:
- gave numbers to parts that had none: 5
Connections:
- net +5C: now reaches C1401.1, SW1401.2 (B), U1401.3 (VI)
- net 3V3 renamed +3V3
Other:
- moved on the sheet: BT1401, C1401, C1402, SW1401, U1401

Commit message: DRC pass
Connections:
- net +3V3 renamed Vdd2
Changed lines of the file:
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@@
     (stroke (width 0) (type default) (color 0 0 0 0))
+  )
+  (hierarchical_label "Vdd2" (shape input) (at 161.29 52.07 0)
+    (effects (font (size 1.27 1.27)) (justify left))
   )
   (symbol (lib_id "Regulator_Linear:MCP1700-3302E_SOT23") (at 138.43 52.07 0) (unit 1)
@@
       (effects (font (size 1.27 1.27)) hide)
     )
-    (pin "1")
-  )
-  (symbol (lib_id "power:+3V3") (at 161.29 52.07 0) (unit 1)
-    (in_bom yes) (on_board yes) (fields_autoplaced)
-    (property "Reference" "#PWR0119" (id 0) (at 161.29 55.88 0)
-      (effects (font (size 1.27 1.27)) hide)
-    )
-    (property "Value" "+3V3" (id 1) (at 161.29 48.4942 0))
-    (property "Footprint" "" (id 2) (at 161.29 52.07 0)
-      (effects (font (size 1.27 1.27)) hide)
-    )
-    (property "Datasheet" "" (id 3) (at 161.29 52.07 0)
-      (effects (font (size 1.27 1.27)) hide)
-    )

Commit message: DRC OK
Parts:
- removed U1401: MCP1700-3302E_SOT23, Package_TO_SOT_SMD:SOT-23, symbol Regulator_Linear:MCP1700-3302E_SOT23
- added U1402: MCP1700x-330xxTT, Package_TO_SOT_SMD:SOT-23, symbol Regulator_Linear:MCP1700x-330xxTT
Connections:
- net +5C: now also U1402.3 (VI)
- net GND2: now also U1402.1 (GND)
- net Vdd2: now also U1402.2 (VO)
