File: pcb/Tail_D.kicad_sch (KiCad schematic)
At the start: 8 parts

Commit message: Corrections to the coax driver
Changed lines of the file:
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@@
     (effects (font (size 1.27 1.27)) (justify left))
   )
-  (symbol (lib_id "power:GND2") (at 140.97 88.9 0)
+  (symbol (lib_id "power:GND2") (at 140.97 88.9 0) (unit 1)
     (in_bom yes) (on_board yes)
     (property "Reference" "#PWR?" (id 0) (at 140.97 95.25 0)
@@
     (pin "1")
   )
-  (symbol (lib_id "Connector:Conn_Coaxial") (at 115.57 110.49 0) (mirror y)
+  (symbol (lib_id "Connector:Conn_Coaxial") (at 115.57 110.49 0) (mirror y) (unit 1)
     (in_bom yes) (on_board yes)
     (property "Reference" "J?" (id 0) (at 113.03 111.125 0)
@@
     (pin "2")
   )
-  (symbol (lib_id "Device:R") (at 156.21 110.49 270)
+  (symbol (lib_id "Device:R") (at 156.21 110.49 270) (unit 1)
     (in_bom yes) (on_board yes)
     (property "Reference" "R?" (id 0) (at 157.3784 112.268 0)
@@
     (pin "2")
   )
-  (symbol (lib_id "power:GND2") (at 140.97 129.54 0)
+  (symbol (lib_id "power:GND2") (at 140.97 129.54 0) (unit 1)
     (in_bom yes) (on_board yes)
     (property "Reference" "#PWR?" (id 0) (at 140.97 135.89 0)
@@
     (pin "1")
   )
-  (symbol (lib_id "Connector:Conn_Coaxial") (at 114.3 69.85 0) (mirror y)
+  (symbol (lib_id "Connector:Conn_Coaxial") (at 114.3 69.85 0) (mirror y) (unit 1)
     (in_bom yes) (on_board yes)
     (property "Reference" "J?" (id 0) (at 111.76 70.485 0)
@@
     (pin "2")
   )
-  (symbol (lib_id "CoaxTester:LTV-817") (at 129.54 72.39 0) (mirror y)
+  (symbol (lib_id "CoaxTester:LTV-817") (at 129.54 72.39 0) (mirror y) (unit 1)
     (in_bom yes) (on_board yes)
     (property "Reference" "U?" (id 0) (at 129.54 61.849 0))
@@
     (pin "4")
   )
-  (symbol (lib_id "Device:R") (at 156.21 69.85 270)
+  (symbol (lib_id "Device:R") (at 156.21 69.85 270) (unit 1)
     (in_bom yes) (on_board yes)
     (property "Reference" "R?" (id 0) (at 157.3784 71.628 0)
@@
     (pin "2")
   )
-  (symbol (lib_id "Device:R") (at 148.59 80.01 180)
+  (symbol (lib_id "Device:R") (at 148.59 80.01 180) (unit 1)
     (in_bom yes) (on_board yes)
     (property "Reference" "R?" (id 0) (at 146.812 81.1784 0)
@@
     (pin "2")
   )
-  (symbol (lib_id "CoaxTester:LTV-817") (at 129.54 113.03 0) (mirror y)
+  (symbol (lib_id "CoaxTester:LTV-817") (at 129.54 113.03 0) (mirror y) (unit 1)
     (in_bom yes) (on_board yes)
     (property "Reference" "U?" (id 0) (at 129.54 102.489 0))
@@
     (pin "4")
   )
-  (symbol (lib_id "Device:R") (at 148.59 120.65 180)
+  (symbol (lib_id "Device:R") (at 148.59 120.65 180) (unit 1)
     (in_bom yes) (on_board yes)
     (property "Reference" "R?" (id 0) (at 146.812 121.8184 0)

Commit message: Schematic complete
Parts:
- gave numbers to parts that had none: 8
Changed lines of the file:
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@@
   (symbol (lib_id "power:GND2") (at 140.97 88.9 0) (unit 1)
     (in_bom yes) (on_board yes)
-    (property "Reference" "#PWR?" (id 0) (at 140.97 95.25 0)
+    (property "Reference" "#PWR01201" (id 0) (at 140.97 95.25 0)
       (effects (font (size 1.27 1.27)) hide)
     )
@@
   (symbol (lib_id "Connector:Conn_Coaxial") (at 115.57 110.49 0) (mirror y) (unit 1)
     (in_bom yes) (on_board yes)
-    (property "Reference" "J?" (id 0) (at 113.03 111.125 0)
+    (property "Reference" "J1202" (id 0) (at 113.03 111.125 0)
       (effects (font (size 1.27 1.27)) (justify left))
     )
@@
   (symbol (lib_id "Device:R") (at 156.21 110.49 270) (unit 1)
     (in_bom yes) (on_board yes)
-    (property "Reference" "R?" (id 0) (at 157.3784 112.268 0)
+    (property "Reference" "R1204" (id 0) (at 157.3784 112.268 0)
       (effects (font (size 1.27 1.27)) (justify left))
     )
@@
   (symbol (lib_id "power:GND2") (at 140.97 129.54 0) (unit 1)
     (in_bom yes) (on_board yes)
-    (property "Reference" "#PWR?" (id 0) (at 140.97 135.89 0)
+    (property "Reference" "#PWR01202" (id 0) (at 140.97 135.89 0)
       (effects (font (size 1.27 1.27)) hide)
     )
@@
   (symbol (lib_id "Connector:Conn_Coaxial") (at 114.3 69.85 0) (mirror y) (unit 1)
     (in_bom yes) (on_board yes)
-    (property "Reference" "J?" (id 0) (at 111.76 70.485 0)
+    (property "Reference" "J1201" (id 0) (at 111.76 70.485 0)
       (effects (font (size 1.27 1.27)) (justify left))
     )
@@
   (symbol (lib_id "CoaxTester:LTV-817") (at 129.54 72.39 0) (mirror y) (unit 1)
     (in_bom yes) (on_board yes)
-    (property "Reference" "U?" (id 0) (at 129.54 61.849 0))
+    (property "Reference" "U1201" (id 0) (at 129.54 61.849 0))
     (property "Value" "LTV-817" (id 1) (at 129.54 64.1604 0))
     (property "Footprint" "local_opto:LTV_817" (id 2) (at 129.54 66.4718 0)
@@
   (symbol (lib_id "Device:R") (at 156.21 69.85 270) (unit 1)
     (in_bom yes) (on_board yes)
-    (property "Reference" "R?" (id 0) (at 157.3784 71.628 0)
+    (property "Reference" "R1203" (id 0) (at 157.3784 71.628 0)
       (effects (font (size 1.27 1.27)) (justify left))
     )
@@
   (symbol (lib_id "Device:R") (at 148.59 80.01 180) (unit 1)
     (in_bom yes) (on_board yes)
-    (property "Reference" "R?" (id 0) (at 146.812 81.1784 0)
+    (property "Reference" "R1201" (id 0) (at 146.812 81.1784 0)
       (effects (font (size 1.27 1.27)) (justify left))
     )
@@
   (symbol (lib_id "CoaxTester:LTV-817") (at 129.54 113.03 0) (mirror y) (unit 1)
     (in_bom yes) (on_board yes)
-    (property "Reference" "U?" (id 0) (at 129.54 102.489 0))
+    (property "Reference" "U1202" (id 0) (at 129.54 102.489 0))
     (property "Value" "LTV-817" (id 1) (at 129.54 104.8004 0))
     (property "Footprint" "local_opto:LTV_817" (id 2) (at 129.54 107.1118 0)
@@
   (symbol (lib_id "Device:R") (at 148.59 120.65 180) (unit 1)
     (in_bom yes) (on_board yes)
-    (property "Reference" "R?" (id 0) (at 146.812 121.8184 0)
+    (property "Reference" "R1202" (id 0) (at 146.812 121.8184 0)
       (effects (font (size 1.27 1.27)) (justify left))
     )
