File: pcb/CoaxTester.kicad_sch (KiCad schematic)
At the start: 44 parts

Commit message: Schematic complete
Parts:
- removed U?: ATmega88-20AU, Package_QFP:TQFP-32_7x7mm_P0.8mm, symbol MCU_Microchip_ATmega:ATmega88-20AU
- added U101: ATmega88-20A, Package_QFP:TQFP-32_7x7mm_P0.8mm, symbol MCU_Microchip_ATmega:ATmega88-20A
- Lg: renamed from Lg?; value SJM Logo -> logo
- U: renamed from U?; footprint CoaxTester:EA_DOGM128-6 -> Display:EA_DOGM128-6
- gave numbers to parts that had none: 41
Connections:
- net 3V3 is gone; now on net +3.3V: C101.2, C102.1, C104.1, H101.1 (Vcc)
- net DIN0: now also U101.2 (PD4)
- net DIN1: now also U101.9 (PD5)
- net DIN2: now also U101.10 (PD6)
- net DISP_BKLT: now also U101.26 (PC3)
- net DOUT0: now also U101.23 (PC0)
- net DOUT1: now also U101.24 (PC1)
- net DOUT2: now also U101.25 (PC2)
- net GND: now also U101.21 (GND), U101.3 (GND), U101.5 (GND)
- net MISO: now also U101.16 (PB4)
- net MOSI: now also U101.15 (PB3)
- net SCK: now also U101.17 (PB5)
- net XBEE_DIN: now also U101.31 (PD1)
- net XBEE_DOUT: now also U101.30 (PD0)
- net ~{BKLT}: now also U101.28 (PC5)
- net ~{DISP_CS}: now also U101.14 (PB2)
- net ~{DISP_REST}: now also U101.13 (PB1)
- net ~{RESET}: now also J101.5 (Pin_5), U101.29 (~{RESET}/PC6)
- net ~{START}: now also U101.27 (PC4)
- net ~{XB_RESET}: now also U101.32 (PD2)
- net ~{XB_SLEEP}: now also U101.1 (PD3)
- net at R101.1: now also U101.11 (PD7)
- net +3.3V: now reaches U.1 (A1+)
- net +3.3V: now also U.2 (A2+), U.3 (A3+), U.34 (VDD2), U.35 (VDD), U101.18 (AVCC), U101.4 (VCC), U101.6 (VCC)
- net A0 renamed A0_RW
- net A0_RW: now also U101.7 (XTAL1/PB6)
- net T_3v3 renamed +3V3
- no-connect marks 28 -> 25
Other:
- sheet Tail Power ports: added none; removed 3V3, 5V
- note removed: "The level shifter is specifically for the XBee module which operates at 3V"

Commit message: DRC pass
Parts:
- removed U: EA_DOGM128X-6, Display:EA_DOGM128-6, symbol Display_Graphic:EA_DOGM128X-6
- added U102: EA_DOGM128X-6, Display:EA_DOGM128-6, symbol CoaxTester:EA_DOGM128X-6
Connections:
- net A0_RW: now also U102.38 (A0)
- net GND: now also U102.26 (VSS), U102.33 (VSS)
- net MOSI: now also U102.36 (SI)
- net SCK: now also U102.37 (SCL)
- net ~{DISP_CS}: now also U102.40 (~{CS1B})
- net ~{DISP_REST}: now also U102.39 (~{RST})
- net at C103.2: now also U102.31 (CAP3P)
- net at C106.1: now also U102.29 (CAP1P)
- net at C105.1, C106.2: now also U102.30 (CAP1N)
- net at C113.1: now also U102.24 (V3)
- net at C109.1: now also U102.23 (V2)
- net at C108.1: now also U102.21 (V0)
- net at C110.1: now also U102.25 (V4)
- net at C112.1: now also U102.22 (V1)
- net at U103.2 (OUT), U103.3 (OUT), U103.5 (OUT): now also U102.18 (C1-), U102.19 (C2-), U102.20 (C3-)
- net at C111.1: now also U102.32 (VOUT)
- net at C107.1: now also U102.27 (CAP2N)
- net at C107.2: now also U102.28 (CAP2P)
- net +3.3V renamed Vdd
- net Vdd: now also U102.1 (A1+), U102.2 (A2+), U102.3 (A3+), U102.34 (VDD2), U102.35 (VDD)
- net +3V3 renamed Vdd2
Other:
- sheet Controls ports: added Vdd; removed none
- sheet Head Power ports: added Vdd; removed 3V3
- sheet Head_Line_Driver ports: added Vdd; removed none
- sheet Tail Power ports: added Vdd2; removed none

Commit message: Cleaning up and RC checks
Parts:
- LG?: renamed from LG102; value KiCad Logo -> logo
- LG?: renamed from LG104; value KiCad Logo -> logo
- LG?: renamed from LG103; value SJM Logo -> logo
- renumbered Lg to LG
Changed lines of the file:
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@@
   (symbol (lib_id "mech:logo") (at 201.93 48.26 0) (unit 1)
     (in_bom yes) (on_board yes) (dnp no)
-    (property "Reference" "LG102" (at 201.93 48.26 0)
-      (effects (font (size 1.27 1.27)) hide)
-    )
-    (property "Value" "KiCad Logo" (at 201.93 53.34 0)
+    (property "Reference" "LG?" (at 201.93 48.26 0)
+      (effects (font (size 1.27 1.27)) hide)
+    )
+    (property "Value" "logo" (at 201.93 53.34 0)
       (effects (font (size 1.27 1.27)))
     )
@@
       (project "CoaxTester"
         (path "/9bac9ad3-a7b9-47f0-87c7-d8630653df68"
-          (reference "LG102") (unit 1)
+          (reference "LG?") (unit 1)
         )
       )
@@
   (symbol (lib_id "mech:logo") (at 184.15 48.26 0) (unit 1)
     (in_bom yes) (on_board yes) (dnp no)
-    (property "Reference" "LG101" (at 184.15 48.26 0)
+    (property "Reference" "LG?" (at 184.15 48.26 0)
       (effects (font (size 1.27 1.27)) hide)
     )
@@
       (effects (font (size 1.27 1.27)) hide)
     )
-    (property "Reference" "Lg" (at 184.15 48.26 0)
+    (property "Reference" "LG" (at 184.15 48.26 0)
       (effects (font (size 1.27 1.27)) hide)
     )
@@
       (project "CoaxTester"
         (path "/9bac9ad3-a7b9-47f0-87c7-d8630653df68"
-          (reference "LG101") (unit 1)
+          (reference "LG?") (unit 1)
         )
       )
@@
   (symbol (lib_id "mech:logo") (at 359.41 48.26 0) (unit 1)
     (in_bom yes) (on_board yes) (dnp no)
-    (property "Reference" "LG104" (at 359.41 48.26 0)
-      (effects (font (size 1.27 1.27)) hide)
-    )
-    (property "Value" "KiCad Logo" (at 359.41 53.34 0)
+    (property "Reference" "LG?" (at 359.41 48.26 0)
+      (effects (font (size 1.27 1.27)) hide)
+    )
+    (property "Value" "logo" (at 359.41 53.34 0)
       (effects (font (size 1.27 1.27)))
     )
@@
       (project "CoaxTester"
         (path "/9bac9ad3-a7b9-47f0-87c7-d8630653df68"
-          (reference "LG104") (unit 1)
+          (reference "LG?") (unit 1)
         )
       )
@@
   (symbol (lib_id "mech:logo") (at 346.71 48.26 0) (unit 1)
     (in_bom yes) (on_board yes) (dnp no)
-    (property "Reference" "LG103" (at 346.71 48.26 0)
-      (effects (font (size 1.27 1.27)) hide)
-    )
-    (property "Value" "SJM Logo" (at 346.71 53.34 0)
+    (property "Reference" "LG?" (at 346.71 48.26 0)
+      (effects (font (size 1.27 1.27)) hide)
+    )
+    (property "Value" "logo" (at 346.71 53.34 0)
       (effects (font (size 1.27 1.27)))
     )
@@
       (project "CoaxTester"
         (path "/9bac9ad3-a7b9-47f0-87c7-d8630653df68"
-          (reference "LG103") (unit 1)
-        )
-      )
+          (reference "LG?") (unit 1)
+        )
+      )
