File: pcb/Controls.kicad_sch (KiCad schematic)
At the start: 11 parts

Commit message: Updates the schematic and fixes some symbols
Parts:
- C? (x2): footprint (none) -> Capacitor_SMD:C_0805_2012Metric
- R? (x4): footprint (none) -> Resistor_SMD:R_0805_2012Metric
- U? (x3): footprint (none) -> Package_SO:SO-16_3.9x9.9mm_P1.27mm
Changed lines of the file:
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@@
       (effects (font (size 1.27 1.27)) (justify left))
     )
-    (property "Footprint" "" (id 2) (at 143.8402 121.92 0)
+    (property "Footprint" "Capacitor_SMD:C_0805_2012Metric" (id 2) (at 143.8402 121.92 0)
       (effects (font (size 1.27 1.27)) hide)
     )
@@
       (effects (font (size 1.27 1.27)) (justify left))
     )
-    (property "Footprint" "" (id 2) (at 129.032 42.545 90)
+    (property "Footprint" "Resistor_SMD:R_0805_2012Metric" (id 2) (at 129.032 42.545 90)
       (effects (font (size 1.27 1.27)) hide)
     )
@@
     (property "Reference" "R?" (id 0) (at 137.16 47.9892 90))
     (property "Value" "470Ω" (id 1) (at 137.16 50.5261 90))
-    (property "Footprint" "" (id 2) (at 137.16 54.483 90)
+    (property "Footprint" "Resistor_SMD:R_0805_2012Metric" (id 2) (at 137.16 54.483 90)
       (effects (font (size 1.27 1.27)) hide)
     )
@@
     (property "Reference" "U?" (id 0) (at 152.4 45.1952 0))
     (property "Value" "74LS14" (id 1) (at 152.4 47.7321 0))
-    (property "Footprint" "" (id 2) (at 152.4 52.705 0)
+    (property "Footprint" "Package_SO:SO-16_3.9x9.9mm_P1.27mm" (id 2) (at 152.4 52.705 0)
       (effects (font (size 1.27 1.27)) hide)
     )
@@
       (effects (font (size 1.27 1.27)) (justify left))
     )
-    (property "Footprint" "" (id 2) (at 129.032 96.52 90)
+    (property "Footprint" "Resistor_SMD:R_0805_2012Metric" (id 2) (at 129.032 96.52 90)
       (effects (font (size 1.27 1.27)) hide)
     )
@@
       (effects (font (size 1.27 1.27)) (justify left))
     )
-    (property "Footprint" "" (id 2) (at 143.8402 67.945 0)
+    (property "Footprint" "Capacitor_SMD:C_0805_2012Metric" (id 2) (at 143.8402 67.945 0)
       (effects (font (size 1.27 1.27)) hide)
     )
@@
     (property "Reference" "U?" (id 0) (at 86.995 145.415 0))
     (property "Value" "74LS14" (id 1) (at 83.185 135.255 0))
-    (property "Footprint" "" (id 2) (at 83.185 135.89 0)
+    (property "Footprint" "Package_SO:SO-16_3.9x9.9mm_P1.27mm" (id 2) (at 83.185 135.89 0)
       (effects (font (size 1.27 1.27)) hide)
     )
@@
     (property "Reference" "U?" (id 0) (at 152.4 99.1702 0))
     (property "Value" "74LS14" (id 1) (at 152.4 101.7071 0))
-    (property "Footprint" "" (id 2) (at 152.4 106.68 0)
+    (property "Footprint" "Package_SO:SO-16_3.9x9.9mm_P1.27mm" (id 2) (at 152.4 106.68 0)
       (effects (font (size 1.27 1.27)) hide)
     )
@@
     (property "Reference" "R?" (id 0) (at 137.16 101.9642 90))
     (property "Value" "470Ω" (id 1) (at 137.16 104.5011 90))
-    (property "Footprint" "" (id 2) (at 137.16 108.458 90)
+    (property "Footprint" "Resistor_SMD:R_0805_2012Metric" (id 2) (at 137.16 108.458 90)
       (effects (font (size 1.27 1.27)) hide)
     )

Commit message: Schematic complete
Parts:
- gave numbers to parts that had none: 7
Connections:
- net 3V3 renamed +3.3V
Other:
- moved on the sheet: C1502, R1501, R1503, SW?, U1501A, U1501G

Commit message: DRC pass
Connections:
- net +3.3V renamed Vdd
Changed lines of the file:
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@@
+    (stroke (width 0) (type default) (color 0 0 0 0))
+  )
+  (wire (pts (xy 123.19 28.194) (xy 130.81 28.194))
     (stroke (width 0) (type default) (color 0 0 0 0))
   )
@@
     (stroke (width 0) (type default) (color 0 0 0 0))
   )
-  (wire (pts (xy 130.81 31.75) (xy 130.81 35.56))
-    (stroke (width 0) (type default) (color 0 0 0 0))
+  (wire (pts (xy 130.81 28.194) (xy 130.81 35.56))
+    (stroke (width 0) (type default) (color 0 0 0 0))
+  )
+  (label "Vdd" (at 82.55 118.11 0)
+    (effects (font (size 1.27 1.27)) (justify left bottom))
+  )
+  (label "Vdd" (at 128.778 28.194 0)
+    (effects (font (size 1.27 1.27)) (justify left bottom))
+  )
+  (label "Vdd" (at 130.81 90.17 0)
+    (effects (font (size 1.27 1.27)) (justify left bottom))
   )
   (hierarchical_label "SW_START" (shape input) (at 165.1 52.07 0)
     (effects (font (size 1.27 1.27)) (justify left))
   )
+  (hierarchical_label "Vdd" (shape input) (at 123.19 28.194 180)
+    (effects (font (size 1.27 1.27)) (justify right))
+  )
   (hierarchical_label "SW_BKLT" (shape input) (at 166.37 106.68 0)
     (effects (font (size 1.27 1.27)) (justify left))
@@
     )
     (property "Datasheet" "" (id 3) (at 142.875 130.175 0)
-      (effects (font (size 1.27 1.27)) hide)
-    )
-    (pin "1")
-  )
-  (symbol (lib_id "power:+3.3V") (at 82.55 118.11 0) (unit 1)
-    (in_bom yes) (on_board yes) (fields_autoplaced)
-    (property "Reference" "#PWR01501" (id 0) (at 82.55 121.92 0)
-      (effects (font (size 1.27 1.27)) hide)
-    )
-    (property "Value" "+3.3V" (id 1) (at 82.55 114.5342 0))
-    (property "Footprint" "" (id 2) (at 82.55 118.11 0)
-      (effects (font (size 1.27 1.27)) hide)
-    )
-    (property "Datasheet" "" (id 3) (at 82.55 118.11 0)
       (effects (font (size 1.27 1.27)) hide)
     )
@@
     (pin "2")
   )
-  (symbol (lib_id "power:+3.3V") (at 130.81 90.17 0) (unit 1)
-    (in_bom yes) (on_board yes) (fields_autoplaced)
-    (property "Reference" "#PWR01505" (id 0) (at 130.81 93.98 0)
-      (effects (font (size 1.27 1.27)) hide)
-    )
-    (property "Value" "+3.3V" (id 1) (at 130.81 86.5942 0))
-    (property "Footprint" "" (id 2) (at 130.81 90.17 0)
-      (effects (font (size 1.27 1.27)) hide)
-    )
-    (property "Datasheet" "" (id 3) (at 130.81 90.17 0)
-      (effects (font (size 1.27 1.27)) hide)
-    )
-    (pin "1")
-  )
   (symbol (lib_id "power:GND") (at 130.81 76.2 0) (unit 1)
     (in_bom yes) (on_board yes) (fields_autoplaced)
@@
     (pin "1")
     (pin "2")
-    (pin "3")
-    (pin "4")
-    (pin "5")
-    (pin "6")
-    (pin "8")
-    (pin "9")
-    (pin "10")
-    (pin "11")
-    (pin "12")
-    (pin "13")
-    (pin "14")
-    (pin "7")
   )
   (symbol (lib_id "Device:R") (at 130.81 96.52 0) (unit 1)
@@
       (effects (font (size 1.27 1.27)) hide)
     )
-    (pin "1")
-    (pin "2")
-    (pin "3")
-    (pin "4")
-    (pin "5")
-    (pin "6")
-    (pin "8")
-    (pin "9")
-    (pin "10")
-    (pin "11")
-    (pin "12")
-    (pin "13")
     (pin "14")
     (pin "7")
@@
       (effects (font (size 1.27 1.27)) hide)
     )
-    (pin "1")
-    (pin "2")
     (pin "3")
     (pin "4")
-    (pin "5")
-    (pin "6")
-    (pin "8")
-    (pin "9")
-    (pin "10")
-    (pin "11")
-    (pin "12")
-    (pin "13")
-    (pin "14")
-    (pin "7")
-  )
-  (symbol (lib_id "power:+3.3V") (at 130.81 31.75 0) (unit 1)
-    (in_bom yes) (on_board yes) (fields_autoplaced)
-    (property "Reference" "#PWR01503" (id 0) (at 130.81 35.56 0)
-      (effects (font (size 1.27 1.27)) hide)
-    )
-    (property "Value" "+3.3V" (id 1) (at 130.81 28.1742 0))
-    (property "Footprint" "" (id 2) (at 130.81 31.75 0)
-      (effects (font (size 1.27 1.27)) hide)
-    )
-    (property "Datasheet" "" (id 3) (at 130.81 31.75 0)
-      (effects (font (size 1.27 1.27)) hide)
-    )
-    (pin "1")
   )
   (symbol (lib_id "Device:R") (at 137.16 106.68 90) (unit 1)

Commit message: DRC OK
Parts:
- added unit 5 of U1501
- added unit 4 of U1501
- added unit 3 of U1501
- added unit 6 of U1501
- gave numbers to parts that had none: 2
Connections:
- no-connect marks 0 -> 8
